File: PCB 111000_New/PCB 111000_New.sch (EAGLE design)
At the start: 52 parts, among them IC1 FT230XS, IC2 MEGA8-P, IC3 MEGA8-P, SW1 DPDT, SW2 NO_SW, SW3 NO_PB_1, SW4 NO_PB_1, SW5 NO_PB_1

Commit message: Update PCB 111000_New.sch
Other:
- note added: "USER SWITCHES ARE TOO CLOSE TO THE +5V TRACK"
Changed lines of the file:
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@@
 <text x="-185.42" y="38.1" size="6.35" layer="91">PCB111000_NEW</text>
 <text x="-185.42" y="25.4" size="6.35" layer="91">Uses Common cathode or</text>
+<text x="-187.96" y="-40.64" size="6.4516" layer="91">USER SWITCHES ARE TOO CLOSE TO THE +5V TRACK</text>
 </plain>
 <instances>
